File: simulation/filter.sch (KiCad schematic (older format))
At the start: 16 parts, among them Q1 BS170

Commit message: Playing with some different values for 40m
Parts:
- C6: value 1n -> 330p
- L1: value 600n -> 560n
- L3: value 470n -> 2u
- V1: value 3 -> 2
Connections:
- net GND: now also R2.2; no longer R2.1
- net V4: now also R2.1; no longer R2.2
Changed lines of the file:
@@
 P 4900 4800
 F 0 "V1" H 5128 4846 50  0000 L CNN
-F 1 "3" H 5128 4755 50  0000 L CNN
+F 1 "2" H 5128 4755 50  0000 L CNN
 F 2 "" H 4900 4800 50  0001 C CNN
 F 3 "~" H 4900 4800 50  0001 C CNN
@@
 F 3 "~" H 7550 3550 50  0001 C CNN
 	1    7550 3550
-	-1   0    0    1
+	-1   0    0    -1
 $EndComp
 Wire Wire Line
@@
 Text Notes 3900 5950 0    50   ~ 0
 .control\n* I'm trying to measure power dissipation of the transistor\n* However, this doesn't show up as a graphable signal\nlet Qpower = v(V1) * id(Q1)\nplot Qpower\n.endc
-$Comp
-L Device:C C1
-U 1 1 5EF523A5
-P 5600 3350
-F 0 "C1" V 5348 3350 50  0000 C CNN
-F 1 "1n" V 5439 3350 50  0000 C CNN
-F 2 "" H 5638 3200 50  0001 C CNN
-F 3 "~" H 5600 3350 50  0001 C CNN
-	1    5600 3350
-	0    1    1    0
-$EndComp
 $Comp
 L Device:L L3
@@
 P 4800 3150
 F 0 "L3" H 4853 3196 50  0000 L CNN
-F 1 "470n" H 4853 3105 50  0000 L CNN
+F 1 "2u" H 4853 3105 50  0000 L CNN
 F 2 "" H 4800 3150 50  0001 C CNN
 F 3 "~" H 4800 3150 50  0001 C CNN
@@
 P 6200 3350
 F 0 "L1" V 6019 3350 50  0000 C CNN
-F 1 "600n" V 6110 3350 50  0000 C CNN
+F 1 "560n" V 6110 3350 50  0000 C CNN
 F 2 "" H 6200 3350 50  0001 C CNN
 F 3 "~" H 6200 3350 50  0001 C CNN
@@
 P 5400 3600
 F 0 "C6" H 5285 3554 50  0000 R CNN
-F 1 "1n" H 5285 3645 50  0000 R CNN
+F 1 "330p" H 5285 3645 50  0000 R CNN
 F 2 "" H 5438 3450 50  0001 C CNN
 F 3 "~" H 5400 3600 50  0001 C CNN
@@
 	-1   0    0    1
 $EndComp
+$Comp
+L Device:C C1
+U 1 1 5EF523A5
+P 5600 3350
+F 0 "C1" V 5348 3350 50  0000 C CNN
+F 1 "1n" V 5439 3350 50  0000 C CNN
+F 2 "" H 5638 3200 50  0001 C CNN
+F 3 "~" H 5600 3350 50  0001 C CNN
+	1    5600 3350
+	0    1    1    0
+$EndComp
 $EndSCHEMATC
